File: Corne_holes_mirrored.kicad_pcb (KiCad board)
At the start: 2 copper layers, 133.7 x 91.4 mm, 48 parts, among them J1 MJ-4PP-9, J2 OLED, SW1 SW_PUSH, SW10 SW_PUSH, SW11 SW_PUSH, SW12 SW_PUSH, SW13 SW_PUSH, SW14 SW_PUSH, SW15 SW_PUSH, SW16 SW_PUSH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

Commit message: Fix issues, add step file
Other:
- outline, holes or cut-outs redrawn
- net class Default removed
